File: NodeLoRaGrove.sch (KiCad schematic (older format))
At the start: 42 parts, among them P1 PICKIT PROGRAMMER, P2 USB_A, P3 CONN_01X02, P4 GROVE 2, P5 GROVE 4, P6 GROVE 1, P7 GROVE 3, SW1 SW_PUSH, U1 AP2112, U2 MCP73831T-2ATI/OT, U3 ATmega32U4, Y1 8Mhz

Commit message: Update schematic
Parts:
- removed U3: ATmega32U4, symbol ATmega32U4
- added U3: ATmega32U4-AU, symbol ATmega32U4-AU
- C1, C2, C3, C4, C5, C6, C7, C8, C9: footprint (none) -> Capacitors_SMD:C_0805_HandSoldering
- D2, D3, D4, D6, D7: footprint (none) -> LEDs:LED_0805
- MODULE1: footprint MICROCHIP_RN2483-I/RM095 -> modules:RN2483
- P1: footprint (none) -> Pin_Headers:Pin_Header_Straight_1x05
- P2: footprint (none) -> Connect:USB_Mini-B
- P3: footprint (none) -> Pin_Headers:Pin_Header_Straight_1x02
- P4, P5, P6, P7: footprint (none) -> Pin_Headers:Pin_Header_Straight_1x04
- R1, R10, R11, R12, R13, R14, R2, R3, R5, R6, R7, R8, R9: footprint (none) -> Resistors_SMD:R_0805_HandSoldering
- U2: footprint SOT95P300X145-5N -> (none)
Connections:
- net +3V3: now also U3.14 (VCC), U3.24 (AVCC), U3.34 (VCC), U3.42 (AREF), U3.44 (AVCC)
- net A0: now also U3.36 ((ADC7/TDI)PF7)
- net A1: now also U3.37 ((ADC6/TDO)PF6)
- net A2: now also U3.38 ((ADC5/TMS)PF5)
- net A3: now also U3.39 ((ADC4/TCK)PF4)
- net D13: now also U3.32 ((ICP3/CLK0/OC4A)PC7)
- net D6: now also U3.27 ((T0/OC4D/ADC10)PD7)
- net D9: now also U3.29 ((ADC12/OC1A/~OC4B~/PCINT12)PB5)
- net GND: now also U3.15 (GND), U3.23 (GND), U3.33 ((~HWB~)PE2), U3.35 (GND), U3.43 (GND), U3.5 (UGND)
- net RST: now also U3.13 (RESET)
- net RX_TX: now also U3.20 ((RXD/INT2)PD2)
- net SCL: now also U3.18 ((OC0B/SCL/INT0)PD0)
- net SDA: now also U3.19 ((SDA/INT1)PD1)
- net TX_RX: now also U3.21 ((TXD/INT3)PD3)
- net VCC: now also U3.2 (UVCC), U3.7 (VBUS)
- net at C9.1, Y1.2: now also U3.16 (XTAL2)
- net at C8.1, Y1.1: now also U3.17 (XTAL1)
- net at R12.1: now also U3.3 (D-)
- net at R11.1: now also U3.4 (D+)
- net at C7.1: now also U3.6 (UCAP)

Commit message: Init PCB
Parts:
- A1: footprint (none) -> TIH:GSG-SMA-EDGE
- D1: value ZENERsmall -> MBR120; footprint (none) -> Diodes_SMD:SOD-123
- P4, P5, P6, P7: footprint Pin_Headers:Pin_Header_Straight_1x04 -> Connectors_JST:JST_PH_S4B-PH-K_04x2.00mm_Angled
- SW1: footprint (none) -> TIH:SW_SPST_KMR2
- U1, U2: footprint (none) -> TO_SOT_Packages_SMD:SOT-23-5
- U3: footprint (none) -> Housings_QFP:TQFP-44_10x10mm_Pitch0.8mm
- Y1: footprint (none) -> Crystals:Crystal_HC49-SD_SMD
Changed lines of the file:
@@
 LIBS:contrib
 LIBS:valves
-LIBS:RN2903-I_RM095
 LIBS:theinventorhouse
 LIBS:USB6B1
 LIBS:MCP73831T-2ATI_OT
 LIBS:antena_good
+LIBS:RN2903-I_RM095
 LIBS:NodeLoRaGrove-cache
 EELAYER 25 0
@@
 F 0 "U1" H 1900 6600 60  0000 C CNN
 F 1 "AP2112" H 2250 6050 60  0000 C CNN
-F 2 "" H 2100 6300 60  0001 C CNN
+F 2 "TO_SOT_Packages_SMD:SOT-23-5" H 2100 6300 60  0001 C CNN
 F 3 "" H 2100 6300 60  0000 C CNN
 	1    2100 6300
@@
 F 0 "P6" H 10950 5500 50  0000 C CNN
 F 1 "GROVE 1" V 11050 5250 50  0000 C CNN
-F 2 "Pin_Headers:Pin_Header_Straight_1x04" H 10950 5250 50  0001 C CNN
+F 2 "Connectors_JST:JST_PH_S4B-PH-K_04x2.00mm_Angled" H 10950 5250 50  0001 C CNN
 F 3 "" H 10950 5250 50  0000 C CNN
 	1    10950 5250
@@
 F 0 "Y1" H 7300 2850 50  0000 C CNN
 F 1 "8Mhz" H 7300 2950 50  0000 C CNN
-F 2 "" H 7300 2750 50  0001 C CNN
+F 2 "Crystals:Crystal_HC49-SD_SMD" H 7300 2750 50  0001 C CNN
 F 3 "" H 7300 2750 50  0000 C CNN
 	1    7300 2750
@@
 P 700 5850
 F 0 "D1" H 700 5650 50  0000 C CNN
-F 1 "ZENERsmall" H 700 5750 50  0000 C CNN
-F 2 "" H 700 5850 50  0001 C CNN
+F 1 "MBR120" H 700 5750 50  0000 C CNN
+F 2 "Diodes_SMD:SOD-123" H 700 5850 50  0001 C CNN
 F 3 "" H 700 5850 50  0000 C CNN
 	1    700  5850
@@
 F 0 "U2" H 4764 6359 50  0000 L CNN
 F 1 "MCP73831T-2ATI/OT" H 4727 6259 50  0000 L CNN
-F 2 "" H 4900 6400 50  0001 L CNN
+F 2 "TO_SOT_Packages_SMD:SOT-23-5" H 4900 6400 50  0001 L CNN
 F 3 "SOT-23 Microchip" H 4050 6350 50  0001 L CNN
 F 4 "MCP73831T-2ATI/OT" H 4500 5550 50  0001 L CNN "MP"
@@
 F 0 "SW1" H 5000 1510 50  0000 C CNN
 F 1 "SW_PUSH" H 4850 1320 50  0000 C CNN
-F 2 "" H 4850 1400 50  0001 C CNN
+F 2 "TIH:SW_SPST_KMR2" H 4850 1400 50  0001 C CNN
 F 3 "" H 4850 1400 50  0000 C CNN
 	1    4850 1400
@@
 F 0 "P7" H 10950 6500 50  0000 C CNN
 F 1 "GROVE 3" V 11050 6250 50  0000 C CNN
-F 2 "Pin_Headers:Pin_Header_Straight_1x04" H 10950 6250 50  0001 C CNN
+F 2 "Connectors_JST:JST_PH_S4B-PH-K_04x2.00mm_Angled" H 10950 6250 50  0001 C CNN
 F 3 "" H 10950 6250 50  0000 C CNN
 	1    10950 6250
@@
 F 0 "P4" H 9750 5500 50  0000 C CNN
 F 1 "GROVE 2" V 9850 5250 50  0000 C CNN
-F 2 "Pin_Headers:Pin_Header_Straight_1x04" H 9750 5250 50  0001 C CNN
+F 2 "Connectors_JST:JST_PH_S4B-PH-K_04x2.00mm_Angled" H 9750 5250 50  0001 C CNN
 F 3 "" H 9750 5250 50  0000 C CNN
 	1    9750 5250
@@
 F 0 "P5" H 9750 6500 50  0000 C CNN
 F 1 "GROVE 4" V 9850 6250 50  0000 C CNN
-F 2 "Pin_Headers:Pin_Header_Straight_1x04" H 9750 6250 50  0001 C CNN
+F 2 "Connectors_JST:JST_PH_S4B-PH-K_04x2.00mm_Angled" H 9750 6250 50  0001 C CNN
 F 3 "" H 9750 6250 50  0000 C CNN
 	1    9750 6250
@@
 F 0 "A1" H 1600 950 60  0000 C CNN
 F 1 "ANT" H 1600 550 60  0000 C CNN
-F 2 "" H 1350 550 60  0001 C CNN
+F 2 "TIH:GSG-SMA-EDGE" H 1350 550 60  0001 C CNN
 F 3 "" H 1350 550 60  0000 C CNN
 	1    1350 550
@@
 F 0 "U3" H 8200 3950 50  0000 C CNN
 F 1 "ATmega32U4-AU" H 8450 700 50  0000 C CNN
-F 2 "" H 10300 3350 50  0001 C CNN
+F 2 "Housings_QFP:TQFP-44_10x10mm_Pitch0.8mm" H 10300 3350 50  0001 C CNN
 F 3 "" H 10300 3350 50  0000 C CNN
 	1    9100 2250

Commit message: Update labels and added logo ElectronicCats
Parts:
- D6: value Led_Small -> CHG
- D7: value Led_Small -> DONE
- P3: value CONN_01X02 -> Battery
- P4: value GROVE 2 -> A0
- P5: value GROVE 4 -> D9
- P6: value GROVE 1 -> I2C
- P7: value GROVE 3 -> A2
- R7: value 1K -> 330R
- R8: value R_Small -> 330R
Changed lines of the file:
@@
 P 10950 5250
 F 0 "P6" H 10950 5500 50  0000 C CNN
-F 1 "GROVE 1" V 11050 5250 50  0000 C CNN
+F 1 "I2C" V 11050 5250 50  0000 C CNN
 F 2 "Connectors_JST:JST_PH_S4B-PH-K_04x2.00mm_Angled" H 10950 5250 50  0001 C CNN
 F 3 "" H 10950 5250 50  0000 C CNN
@@
 P 4000 6200
 F 0 "R7" H 4030 6220 50  0000 L CNN
-F 1 "1K" H 4030 6160 50  0000 L CNN
+F 1 "330R" H 4030 6160 50  0000 L CNN
 F 2 "Resistors_SMD:R_0805_HandSoldering" H 4000 6200 50  0001 C CNN
 F 3 "" H 4000 6200 50  0000 C CNN
@@
 P 3700 6200
 F 0 "D6" H 3650 6325 50  0000 L CNN
-F 1 "Led_Small" H 3525 6100 50  0000 L CNN
+F 1 "CHG" H 3525 6100 50  0000 L CNN
 F 2 "LEDs:LED_0805" V 3700 6200 50  0001 C CNN
 F 3 "" V 3700 6200 50  0000 C CNN
@@
 P 6700 6050
 F 0 "P3" H 6700 6200 50  0000 C CNN
-F 1 "CONN_01X02" V 6800 6050 50  0000 C CNN
+F 1 "Battery" V 6800 6050 50  0000 C CNN
 F 2 "Pin_Headers:Pin_Header_Straight_1x02" H 6700 6050 50  0001 C CNN
 F 3 "" H 6700 6050 50  0000 C CNN
@@
 P 3700 6500
 F 0 "D7" H 3650 6625 50  0000 L CNN
-F 1 "Led_Small" H 3525 6400 50  0000 L CNN
+F 1 "DONE" H 3525 6400 50  0000 L CNN
 F 2 "LEDs:LED_0805" V 3700 6500 50  0001 C CNN
 F 3 "" V 3700 6500 50  0000 C CNN
@@
 P 4000 6500
 F 0 "R8" H 4030 6520 50  0000 L CNN
-F 1 "R_Small" H 4030 6460 50  0000 L CNN
+F 1 "330R" H 4030 6460 50  0000 L CNN
 F 2 "Resistors_SMD:R_0805_HandSoldering" H 4000 6500 50  0001 C CNN
 F 3 "" H 4000 6500 50  0000 C CNN
@@
 P 10950 6250
 F 0 "P7" H 10950 6500 50  0000 C CNN
-F 1 "GROVE 3" V 11050 6250 50  0000 C CNN
+F 1 "A2" V 11050 6250 50  0000 C CNN
 F 2 "Connectors_JST:JST_PH_S4B-PH-K_04x2.00mm_Angled" H 10950 6250 50  0001 C CNN
 F 3 "" H 10950 6250 50  0000 C CNN
@@
 P 9750 5250
 F 0 "P4" H 9750 5500 50  0000 C CNN
-F 1 "GROVE 2" V 9850 5250 50  0000 C CNN
+F 1 "A0" V 9850 5250 50  0000 C CNN
 F 2 "Connectors_JST:JST_PH_S4B-PH-K_04x2.00mm_Angled" H 9750 5250 50  0001 C CNN
 F 3 "" H 9750 5250 50  0000 C CNN
@@
 P 9750 6250
 F 0 "P5" H 9750 6500 50  0000 C CNN
-F 1 "GROVE 4" V 9850 6250 50  0000 C CNN
+F 1 "D9" V 9850 6250 50  0000 C CNN
 F 2 "Connectors_JST:JST_PH_S4B-PH-K_04x2.00mm_Angled" H 9750 6250 50  0001 C CNN
 F 3 "" H 9750 6250 50  0000 C CNN

Commit message: Update Schematic remove leds
Notes and leds remove
Parts:
- removed D2: Led, LEDs:LED_0805, symbol Led_Small
- removed R1: 100R, Resistors_SMD:R_0805_HandSoldering, symbol R_Small
- added P2: ICSP, Pin_Headers:Pin_Header_Straight_2x03, symbol CONN_02X03
- renumbered D4 to D2, D6 to D3, D7 to D4, D3 to D5, P2 to P3, P3 to P4, P4 to P5, P5 to P6, P6 to P7, P7 to P8, R3 to R1, R12 to R10, R13 to R11, R14 to R12, R5 to R2, R6 to R3, R7 to R4, R8 to R5, R2 to R6, R9 to R7, R10 to R8, R11 to R9
Connections:
- net GND: now also P2.1 (P1)
- net RST: now also P2.2 (P2)
- net VCC: now also P2.5 (P5)
- net MOSI: now reaches U3.10 ((PDI/MOSI/PCINT2)PB2)
- net MOSI: now also P2.3 (P3)
- net MISO: now reaches U3.11 ((PDO/MISO/PCINT3)PB3)
- net MISO: now also P2.6 (P6)
- net SCK: now reaches U3.9 ((SCLK/PCINT1)PB1)
- net SCK: now also P2.4 (P4)
- no-connect marks 33 -> 31
Other:
- note removed: "REVISION 2 Analogicos o interrupciones o PWM?"
- moved on the sheet: D5, R6

Commit message: Change USB connector
Parts:
- MODULE1: footprint modules:RN2483 -> TIH:RN2483
- P3: footprint Connect:USB_Mini-B -> TIH:10118192-0001LF

Commit message: Fix Skilcreen
Parts:
- D5: symbol LED -> LED-RESCUE-NodeLoRaGrove
- P3: symbol USB_A -> USB_A-RESCUE-NodeLoRaGrove
- U3: symbol ATmega32U4-AU -> ATmega32U4-AU-RESCUE-NodeLoRaGrove
Changed lines of the file:
@@
 EESchema Schematic File Version 2
+LIBS:NodeLoRaGrove-rescue
 LIBS:power
 LIBS:device
@@
 $EndComp
 $Comp
-L USB_A P3
+L USB_A-RESCUE-NodeLoRaGrove P3
 U 1 1 57D06EF4
 P 6150 1600
@@
 $EndComp
 $Comp
-L LED D5
+L LED-RESCUE-NodeLoRaGrove D5
 U 1 1 57D3ECB0
 P 4950 2600
@@
 NoConn ~ 1450 3150
 $Comp
-L ATmega32U4-AU U3
+L ATmega32U4-AU-RESCUE-NodeLoRaGrove U3
 U 1 1 57D4956F
 P 9100 2250

Commit message: added bom
Parts:
- A1: manf# (none) -> CONSMA003.062
- C1, C2, C6: manf# (none) -> GRM21BR61A106KE19L
- C3, C7: manf# (none) -> GRM21BR71C105KA01L
- C4, C5: manf# (none) -> GRM21BR71E104KA01L
- C8, C9: manf# (none) -> 885012007012
- D1: manf# (none) -> NRVB120VLSFT1G
- D2, D5: manf# (none) -> LTST-C170TBKT
- D3: manf# (none) -> LTST-C170KRKT
- D4: manf# (none) -> SM0805GCL
- MODULE1: manf# (none) -> RN2903-I/RM095
- P3: manf# (none) -> 105017-0001
- R1: manf# (none) -> ESR10EZPJ101
- R10, R9: manf# (none) -> BLM21PG220SN1D
- R11, R12: manf# (none) -> RG2012P-472-B-T5
- R2: manf# (none) -> WR08X1003FTL
- R3, R7, R8: manf# (none) -> CPF0805B10KE1
- R4, R5, R6: manf# (none) -> ESR10EZPF3300
- SW1: manf# (none) -> KMR211G LFS
- U1: manf# (none) -> AP2112K-3.3TRG1
- U2: manf# (none) -> MCP73831T-2DCI/OT
- U3: manf# (none) -> ATMEGA32U2-AU
- Y1: manf# (none) -> HC49SSDLF-8.00MHz
Changed lines of the file:
@@
 LIBS:contrib
 LIBS:valves
-LIBS:theinventorhouse
 LIBS:USB6B1
 LIBS:MCP73831T-2ATI_OT
-LIBS:antena_good
 LIBS:RN2903-I_RM095
 LIBS:NodeLoRaGrove-cache
@@
 F 7 "RN2483-I/RM095" H 2250 2150 50  0001 L CNN "MP"
 F 8 "Bad" H 2250 2150 50  0001 L CNN "Availability"
+F 9 "RN2903-I/RM095" H 2250 2150 60  0001 C CNN "manf#"
 	1    2250 2150
 	1    0    0    -1
@@
 F 2 "TO_SOT_Packages_SMD:SOT-23-5" H 2100 6300 60  0001 C CNN
 F 3 "" H 2100 6300 60  0000 C CNN
+F 4 "AP2112K-3.3TRG1" H 2100 6300 60  0001 C CNN "manf#"
 	1    2100 6300
 	1    0    0    -1
@@
 F 2 "TIH:10118192-0001LF" V 6100 1500 50  0001 C CNN
 F 3 "" V 6100 1500 50  0000 C CNN
+F 4 "105017-0001" H 6150 1600 60  0001 C CNN "manf#"
 	1    6150 1600
 	0    -1   1    0
@@
 F 2 "Crystals:Crystal_HC49-SD_SMD" H 7300 2750 50  0001 C CNN
 F 3 "" H 7300 2750 50  0000 C CNN
+F 4 "HC49SSDLF-8.00MHz" H 7300 2750 60  0001 C CNN "manf#"
 	1    7300 2750
 	0    1    1    0
@@
 F 2 "Capacitors_SMD:C_0805_HandSoldering" H 7100 2550 50  0001 C CNN
 F 3 "" H 7100 2550 50  0000 C CNN
+F 4 "885012007012" H 7100 2550 60  0001 C CNN "manf#"
 	1    7100 2550
 	0    1    1    0
@@
 F 2 "Capacitors_SMD:C_0805_HandSoldering" H 7100 2950 50  0001 C CNN
 F 3 "" H 7100 2950 50  0000 C CNN
+F 4 "885012007012" H 7100 2950 60  0001 C CNN "manf#"
 	1    7100 2950
 	0    1    1    0
@@
 F 2 "Capacitors_SMD:C_0805_HandSoldering" H 7050 1950 50  0001 C CNN
 F 3 "" H 7050 1950 50  0000 C CNN
+F 4 "GRM21BR71C105KA01L" H 7050 1950 60  0001 C CNN "manf#"
 	1    7050 1950
 	1    0    0    -1
@@
 F 2 "Resistors_SMD:R_0805_HandSoldering" V 7430 1500 50  0001 C CNN
 F 3 "" H 7500 1500 50  0000 C CNN
+F 4 "BLM21PG220SN1D" V 7500 1500 60  0001 C CNN "manf#"
 	1    7500 1500
 	0    1    1    0
@@
 F 2 "Resistors_SMD:R_0805_HandSoldering" V 7430 1600 50  0001 C CNN
 F 3 "" H 7500 1600 50  0000 C CNN
+F 4 "BLM21PG220SN1D" V 7500 1600 60  0001 C CNN "manf#"
 	1    7500 1600
 	0    1    1    0
@@
 F 2 "Resistors_SMD:R_0805_HandSoldering" H 1450 6300 50  0001 C CNN
 F 3 "" H 1450 6300 50  0000 C CNN
+F 4 "WR08X1003FTL" H 1450 6300 60  0001 C CNN "manf#"
 	1    1450 6300
 	0    1    1    0
@@
 F 2 "Capacitors_SMD:C_0805_HandSoldering" H 1000 6250 50  0001 C CNN
 F 3 "" H 1000 6250 50  0000 C CNN
+F 4 "GRM21BR61A106KE19L" H 1000 6250 60  0001 C CNN "manf#"
 	1    1000 6250
 	1    0    0    -1
@@
 F 2 "Capacitors_SMD:C_0805_HandSoldering" H 2800 6250 50  0001 C CNN
 F 3 "" H 2800 6250 50  0000 C CNN
+F 4 "GRM21BR61A106KE19L" H 2800 6250 60  0001 C CNN "manf#"
 	1    2800 6250
 	1    0    0    -1
@@
 F 2 "Diodes_SMD:SOD-123" H 700 5850 50  0001 C CNN
 F 3 "" H 700 5850 50  0000 C CNN
+F 4 "NRVB120VLSFT1G" H 700 5850 60  0001 C CNN "manf#"
 	1    700  5850
 	0    -1   -1   0
@@
 F 2 "Resistors_SMD:R_0805_HandSoldering" H 6050 6300 50  0001 C CNN
 F 3 "" H 6050 6300 50  0000 C CNN
+F 4 "CPF0805B10KE1" H 6050 6300 60  0001 C CNN "manf#"
 	1    6050 6300
 	1    0    0    -1
@@
 F 7 "Microchip" H 4100 5550 50  0001 L CNN "MF"
 F 8 "0.48 USD" H 4350 6250 50  0001 L CNN "Price"
+F 9 "MCP73831T-2DCI/OT" H 4950 6000 60  0001 C CNN "manf#"
 	1    4950 6000
 	1    0    0    -1
@@
 F 2 "Resistors_SMD:R_0805_HandSoldering" H 4000 6200 50  0001 C CNN
 F 3 "" H 4000 6200 50  0000 C CNN
+F 4 "ESR10EZPF3300" H 4000 6200 60  0001 C CNN "manf#"
 	1    4000 6200
 	0    1    1    0
@@
 F 2 "LEDs:LED_0805" V 3700 6200 50  0001 C CNN
 F 3 "" V 3700 6200 50  0000 C CNN
+F 4 "LTST-C170KRKT" H 3700 6200 60  0001 C CNN "manf#"
 	1    3700 6200
 	-1   0    0    1
@@
 F 2 "LEDs:LED_0805" V 3700 6500 50  0001 C CNN
 F 3 "" V 3700 6500 50  0000 C CNN
+F 4 "SM0805GCL" H 3700 6500 60  0001 C CNN "manf#"
 	1    3700 6500
 	1    0    0    -1
@@
 F 2 "Resistors_SMD:R_0805_HandSoldering" H 4000 6500 50  0001 C CNN
 F 3 "" H 4000 6500 50  0000 C CNN
+F 4 "ESR10EZPF3300" H 4000 6500 60  0001 C CNN "manf#"
 	1    4000 6500
 	0    1    1    0
@@
 F 2 "Capacitors_SMD:C_0805_HandSoldering" H 6250 6250 50  0001 C CNN
 F 3 "" H 6250 6250 50  0000 C CNN
+F 4 "GRM21BR61A106KE19L" H 6250 6250 60  0001 C CNN "manf#"
 	1    6250 6250
 	1    0    0    -1
@@
 F 2 "Resistors_SMD:R_0805_HandSoldering" H 8450 5600 50  0001 C CNN
 F 3 "" H 8450 5600 50  0000 C CNN
+F 4 "RG2012P-472-B-T5" H 8450 5600 60  0001 C CNN "manf#"
 	1    8450 5600
 	1    0    0    -1
@@
 F 2 "Resistors_SMD:R_0805_HandSoldering" H 8200 5600 50  0001 C CNN
 F 3 "" H 8200 5600 50  0000 C CNN
+F 4 "RG2012P-472-B-T5" H 8200 5600 60  0001 C CNN "manf#"
 	1    8200 5600
 	1    0    0    -1
@@
 F 2 "TIH:SW_SPST_KMR2" H 4850 1400 50  0001 C CNN
 F 3 "" H 4850 1400 50  0000 C CNN
+F 4 "KMR211G LFS" H 4850 1400 60  0001 C CNN "manf#"
 	1    4850 1400
 	1    0    0    -1
@@
 F 2 "Resistors_SMD:R_0805_HandSoldering" H 5300 1150 50  0001 C CNN
 F 3 "" H 5300 1150 50  0000 C CNN
+F 4 "CPF0805B10KE1" H 5300 1150 60  0001 C CNN "manf#"
 	1    5300 1150
 	1    0    0    -1
@@
 Connection ~ 1250 6100
 Wire Wire Line
-	800  6150 800  6100
-Connection ~ 800  6100
-Wire Wire Line
 	1000 6150 1000 6100
 Connection ~ 1000 6100
@@
 F 2 "Resistors_SMD:R_0805_HandSoldering" H 3650 2550 50  0001 C CNN
 F 3 "" H 3650 2550 50  0000 C CNN
+F 4 "CPF0805B10KE1" H 3650 2550 60  0001 C CNN "manf#"
 	1    3650 2550
 	1    0    0    -1
@@
 F 2 "Capacitors_SMD:C_0805_HandSoldering" H 3450 1050 50  0001 C CNN
 F 3 "" H 3450 1050 50  0000 C CNN
+F 4 "GRM21BR71E104KA01L" H 3450 1050 60  0001 C CNN "manf#"
 	1    3450 1050
 	1    0    0    -1
@@
 F 2 "Resistors_SMD:R_0805_HandSoldering" H 1200 2250 50  0001 C CNN
 F 3 "" H 1200 2250 50  0000 C CNN
+F 4 "ESR10EZPJ101" H 1200 2250 60  0001 C CNN "manf#"
 	1    1200 2250
 	1    0    0    -1
@@
 F 2 "LEDs:LED_0805" V 1200 2550 50  0001 C CNN
 F 3 "" V 1200 2550 50  0000 C CNN
+F 4 "LTST-C170TBKT" H 1200 2550 60  0001 C CNN "manf#"
 	1    1200 2550
 	0    -1   -1   0
@@
 F 2 "Capacitors_SMD:C_0805_HandSoldering" H 3850 1050 50  0001 C CNN
 F 3 "" H 3850 1050 50  0000 C CNN
+F 4 "GRM21BR71E104KA01L" H 3850 1050 60  0001 C CNN "manf#"
 	1    3850 1050
 	1    0    0    -1
@@
 F 2 "TIH:GSG-SMA-EDGE" H 1350 550 60  0001 C CNN
 F 3 "" H 1350 550 60  0000 C CNN
+F 4 "CONSMA003.062" H 1350 550 60  0001 C CNN "manf#"
 	1    1350 550
 	-1   0    0    1
@@
 F 2 "Capacitors_SMD:C_0805_HandSoldering" H 2950 6250 50  0001 C CNN
 F 3 "" H 2950 6250 50  0000 C CNN
+F 4 "GRM21BR71C105KA01L" H 2950 6250 60  0001 C CNN "manf#"
 	1    2950 6250
 	1    0    0    -1
@@
 F 2 "LEDs:LED_0805" H 4950 2600 50  0001 C CNN
 F 3 "" H 4950 2600 50  0000 C CNN
+F 4 "LTST-C170TBKT" H 4950 2600 60  0001 C CNN "manf#"
 	1    4950 2600
 	0    -1   -1   0
@@
 F 2 "Resistors_SMD:R_0805_HandSoldering" H 4950 2200 50  0001 C CNN
 F 3 "" H 4950 2200 50  0000 C CNN
+F 4 "ESR10EZPF3300" H 4950 2200 60  0001 C CNN "manf#"
 	1    4950 2200
 	1    0    0    -1
@@
 F 2 "Housings_QFP:TQFP-44_10x10mm_Pitch0.8mm" H 10300 3350 50  0001 C CNN
 F 3 "" H 10300 3350 50  0000 C CNN
+F 4 "ATMEGA32U2-AU" H 9100 2250 60  0001 C CNN "manf#"
 	1    9100 2250
 	1    0    0    -1
